File: LPC1114-dev-board/LPC1114-dev-board.sch (KiCad schematic (older format))
At the start: 59 parts, among them CON1 DC IN, K1 PWR_SEL, P1 CONN_12, P2 SWD, P3 ISP/SERIAL, P4 CONN_12, P5 PROG_RESET, SW1 RESET, SW2 MODE_ISP, U1 LM317T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

Commit message: Move power selection jumper after regulator
Begin Version 1.1 changes
Move power selection jumper after regulator
Connections:
- net labels added: Vreg
- wire segments 188 -> 186
Other:
- note added: "1-2 regulated power\n2-3 JTAG/serial power input"
- moved on the sheet: CON1, K1
Changed lines of the file:
@@
 Sheet 1 1
 Title "LPC 1114 Dev Board"
-Date "1 jun 2014"
-Rev "1.0"
+Date "15 jun 2014"
+Rev "1.1"
 Comp ""
 Comment1 ""
@@
 L BARREL_JACK CON1
 U 1 1 53382859
-P 950 3550
-F 0 "CON1" H 950 3800 60  0000 C CNN
-F 1 "DC IN" H 900 3350 60  0000 C CNN
-F 2 "BARREL_JACK" H 950 3550 60  0000 C CNN
-F 3 "" H 950 3550 60  0000 C CNN
-	1    950  3550
+P 4250 1200
+F 0 "CON1" H 4250 1450 60  0000 C CNN
+F 1 "DC IN" H 4200 1000 60  0000 C CNN
+F 2 "BARREL_JACK" H 4200 900 60  0000 C CNN
+F 3 "" H 4250 1200 60  0000 C CNN
+	1    4250 1200
 	1    0    0    -1
 $EndComp
@@
 Text GLabel 8450 4050 2    30   Input ~ 0
 PROG_VCC
-Text GLabel 2150 3550 3    30   Input ~ 0
+Text GLabel 3450 1300 3    30   Input ~ 0
 PROG_VCC
 $Comp
@@
 L GND #PWR08
 U 1 1 53383FFD
-P 1450 3800
-F 0 "#PWR08" H 1450 3800 30  0001 C CNN
-F 1 "GND" H 1450 3730 30  0000 C CNN
-F 2 "" H 1450 3800 60  0000 C CNN
-F 3 "" H 1450 3800 60  0000 C CNN
-	1    1450 3800
+P 4750 1450
+F 0 "#PWR08" H 4750 1450 30  0001 C CNN
+F 1 "GND" H 4750 1380 30  0000 C CNN
+F 2 "" H 4750 1450 60  0000 C CNN
+F 3 "" H 4750 1450 60  0000 C CNN
+	1    4750 1450
 	1    0    0    -1
 $EndComp
@@
 L CONN_3 K1
 U 1 1 533840B3
-P 2050 3000
-F 0 "K1" V 2000 3000 50  0000 C CNN
-F 1 "PWR_SEL" V 2100 3000 40  0000 C CNN
-F 2 "PIN_ARRAY_3X1" V 2200 3000 60  0000 C CNN
-F 3 "" H 2050 3000 60  0000 C CNN
-	1    2050 3000
+P 3350 800
+F 0 "K1" V 3300 800 50  0000 C CNN
+F 1 "PWR_SEL" V 3400 800 40  0000 C CNN
+F 2 "PIN_ARRAY_3X1" V 3500 800 60  0000 C CNN
+F 3 "" H 3350 800 60  0000 C CNN
+	1    3350 800
 	0    -1   -1   0
 $EndComp
@@
 L +3.3V #PWR023
 U 1 1 533889A9
-P 3050 1050
-F 0 "#PWR023" H 3050 1010 30  0001 C CNN
-F 1 "+3.3V" H 3050 1160 30  0000 C CNN
-F 2 "" H 3050 1050 60  0000 C CNN
-F 3 "" H 3050 1050 60  0000 C CNN
-	1    3050 1050
-	1    0    0    -1
+P 3350 1500
+F 0 "#PWR023" H 3350 1460 30  0001 C CNN
+F 1 "+3.3V" H 3350 1610 30  0000 C CNN
+F 2 "" H 3350 1500 60  0000 C CNN
+F 3 "" H 3350 1500 60  0000 C CNN
+	1    3350 1500
+	-1   0    0    1
 $EndComp
 $Comp
 L VIN #PWR024
 U 1 1 53388BE0
-P 1850 3650
-F 0 "#PWR024" H 1850 3610 30  0001 C CNN
-F 1 "VIN" H 1850 3760 30  0000 C CNN
-F 2 "" H 1850 3650 60  0000 C CNN
-F 3 "" H 1850 3650 60  0000 C CNN
-	1    1850 3650
+P 5250 950
+F 0 "#PWR024" H 5250 910 30  0001 C CNN
+F 1 "VIN" H 5250 1060 30  0000 C CNN
+F 2 "" H 5250 950 60  0000 C CNN
+F 3 "" H 5250 950 60  0000 C CNN
+	1    5250 950
 	1    0    0    -1
 $EndComp
@@
 Connection ~ 1650 1600
 Wire Wire Line
-	2050 1250 3050 1250
+	2050 1250 3250 1250
 Wire Wire Line
 	2250 1250 2250 1750
@@
 	2250 2250 2250 2150
 Wire Wire Line
-	1250 3650 1450 3650
-Wire Wire Line
-	1450 3550 1450 3800
-Wire Wire Line
-	1450 3550 1250 3550
-Connection ~ 1450 3650
+	4550 1300 4750 1300
+Wire Wire Line
+	4750 1200 4750 1450
+Wire Wire Line
+	4750 1200 4550 1200
+Connection ~ 4750 1300
 Wire Wire Line
 	5900 4250 5900 4500
@@
 	7700 4000 9100 4000
 Wire Wire Line
-	1250 3450 1950 3450
+	4550 1100 5250 1100
 Wire Wire Line
 	1050 1600 1050 1250
@@
 	800  1250 1250 1250
 Wire Wire Line
-	1950 3450 1950 3350
-Wire Wire Line
-	2150 3550 2150 3350
+	5250 1100 5250 950
 Wire Wire Line
 	7050 2400 7150 2400
@@
 Wire Wire Line
 	7300 4400 7200 4400
-Wire Wire Line
-	3050 1250 3050 1050
-Wire Wire Line
-	2050 3700 1850 3700
-Wire Wire Line
-	1850 3700 1850 3650
 Wire Wire Line
 	9100 6400 9100 6350
@@
 	5150 2000 5150 2050
 Wire Wire Line
-	2050 3350 2050 3700
+	3350 1150 3350 1500
+Wire Wire Line
+	3250 1250 3250 1150
+Text Label 2850 1250 0    30   ~ 0
+Vreg
+Wire Wire Line
+	3450 1150 3450 1300
+Text Notes 3600 800  0    30   ~ 0
+1-2 regulated power\n2-3 JTAG/serial power input
 $EndSCHEMATC

Commit message: Cleanup
Clarify pitch of SWD connector
Rework power options
Add PWR/GND header connections
Add power indicator LEDs
Parts:
- removed C7: 0.1uF, c_0805, symbol C
- removed C8: 1uF, c_0805, symbol C
- removed P5: PROG_RESET, PIN_ARRAY_2X1, symbol CONN_2
- removed R18, R33: 0, SM0805, symbol R
- removed U3: 74LVC125, SO14N, symbol 74LS125
- added D? (x2): LED, ~, symbol LED
- added D?: 1N4002, SMX-DIODE, symbol DIODE
- added K?: PWR_SEL, PIN_ARRAY_3X1, symbol CONN_3
- added P?: RTS, PIN_ARRAY_2X1, symbol CONN_2
- added R?: 10K, SM0805, symbol R
- added R? (x2): 160, ~, symbol R
- K1: value PWR_SEL -> REG_PWR
- P2: footprint PIN_ARRAY_5x2_2MM -> PIN_ARRAY_5x2_1_27mm
Connections:
- net labels added: VCC_ISP, VCC_PROG
- net labels removed: RTS
- wire segments 186 -> 184
- no-connect marks 3 -> 1
Other:
- note added: "1-2 DC in\n2-3 ISP power input (assume 5V)"
- note added: "1-2 regulated power\n2-3 JTAG provided power (must be set to 3.3V)"
- note added: "3.3V Logic Levels\nVCC is assumed to be 5V"
- note removed: "1-2 regulated power\n2-3 JTAG/serial power input"
- note removed: "3.3V Logic Levels"
- note removed: "Jumper 1 to 2 to enable\nRESET via RTS line"
- moved on the sheet: R37
